Commit message: Replace src with working version (last week stable)

File: src/diffbot_sim/urdf/leader.urdf.xacro (robot description, xacro)
@@ -91,32 +91,139 @@
     </xacro:inertial_box>
   </link>
-  <!-- SMALL BOX FOR LIDAR DETECTION -->
-  <joint name="lidar_box_joint" type="fixed">
-    <parent link="chassis"/>
-    <child link="lidar_box"/>
-    <origin xyz="0 0 0.25" rpy="0 0 0"/>
-  </joint>
-  <link name="lidar_box">
-    <visual>
-      <geometry>
-        <box size="0.08 0.08 0.08"/>
-      </geometry>
-      <material name="red"/>
-    </visual>
-    <collision>
-      <geometry>
-        <box size="0.08 0.08 0.08"/>
-      </geometry>
-    </collision>
-    <xacro:inertial_box mass="0.1" x="0.08" y="0.08" z="0.08">
-      <origin xyz="0 0 0"/>
-    </xacro:inertial_box>
-  </link>
-  <gazebo reference="lidar_box">
-    <material>Gazebo/Red</material>
-  </gazebo>
   <gazebo reference="chassis">
     <material>Gazebo/Blue</material>
   </gazebo>
-  <!-- REST OF YOUR ORIGINAL FILE CONTINUES UNCHANGED -->
+  <joint name="front_left_wheel_joint" type="continuous">
+    <parent link="base_link"/>
+    <child link="front_left_wheel"/>
+    <origin xyz="${front_wheel_x} ${wheel_offset_y} ${wheel_center_z}" rpy="-${pi/2} 0 0"/>
+    <axis xyz="0 0 1"/>
+  </joint>
+  <link name="front_left_wheel">
+    <visual>
+      <origin xyz="0 0 0" rpy="0 0 0"/>
+      <geometry>
+        <cylinder radius="${wheel_radius}" length="${wheel_thickness}"/>
+      </geometry>
+      <material name="black"/>
+    </visual>
+    <collision>
+      <origin xyz="0 0 0" rpy="0 0 0"/>
+      <geometry>
+        <cylinder radius="${wheel_radius}" length="${wheel_thickness}"/>
+      </geometry>
+    </collision>
+    <xacro:inertial_cylinder mass="${wheel_mass}" length="${wheel_thickness}" radius="${wheel_radius}">
+      <origin xyz="0 0 0" rpy="0 0 0"/>
+    </xacro:inertial_cylinder>
+  </link>
+  <gazebo reference="front_left_wheel">
+    <material>Gazebo/Black</material>
+  </gazebo>
+  <joint name="front_right_wheel_joint" type="continuous">
+    <parent link="base_link"/>
+    <child link="front_right_wheel"/>
+    <origin xyz="${front_wheel_x} ${-wheel_offset_y} ${wheel_center_z}" rpy="${pi/2} 0 0"/>
+    <axis xyz="0 0 -1"/>
+  </joint>
+  <link name="front_right_wheel">
+    <visual>
+      <origin xyz="0 0 0" rpy="0 0 0"/>
+      <geometry>
+        <cylinder radius="${wheel_radius}" length="${wheel_thickness}"/>
+      </geometry>
+      <material name="black"/>
+    </visual>
+    <collision>
+      <origin xyz="0 0 0" rpy="0 0 0"/>
+      <geometry>
+        <cylinder radius="${wheel_radius}" length="${wheel_thickness}"/>
+      </geometry>
+    </collision>
+    <xacro:inertial_cylinder mass="${wheel_mass}" length="${wheel_thickness}" radius="${wheel_radius}">
+      <origin xyz="0 0 0" rpy="0 0 0"/>
+    </xacro:inertial_cylinder>
+  </link>
+  <gazebo reference="front_right_wheel">
+    <material>Gazebo/Black</material>
+  </gazebo>
+  <joint name="back_left_wheel_joint" type="continuous">
+    <parent link="base_link"/>
+    <child link="back_left_wheel"/>
+    <origin xyz="${back_wheel_x} ${wheel_offset_y} ${wheel_center_z}" rpy="-${pi/2} 0 0"/>
+    <axis xyz="0 0 1"/>
+  </joint>
+  <link name="back_left_wheel">
+    <visual>
+      <origin xyz="0 0 0" rpy="0 0 0"/>
+      <geometry>
+        <cylinder radius="${wheel_radius}" length="${wheel_thickness}"/>
+      </geometry>
+      <material name="black"/>
+    </visual>
+    <collision>
+      <origin xyz="0 0 0" rpy="0 0 0"/>
+      <geometry>
+        <cylinder radius="${wheel_radius}" length="${wheel_thickness}"/>
+      </geometry>
+    </collision>
+    <xacro:inertial_cylinder mass="${wheel_mass}" length="${wheel_thickness}" radius="${wheel_radius}">
+      <origin xyz="0 0 0" rpy="0 0 0"/>
+    </xacro:inertial_cylinder>
+  </link>
+  <gazebo reference="back_left_wheel">
+    <material>Gazebo/Black</material>
+  </gazebo>
+  <joint name="back_right_wheel_joint" type="continuous">
+    <parent link="base_link"/>
+    <child link="back_right_wheel"/>
+    <origin xyz="${back_wheel_x} ${-wheel_offset_y} ${wheel_center_z}" rpy="${pi/2} 0 0"/>
+    <axis xyz="0 0 -1"/>
+  </joint>
+  <link name="back_right_wheel">
+    <visual>
+      <origin xyz="0 0 0" rpy="0 0 0"/>
+      <geometry>
+        <cylinder radius="${wheel_radius}" length="${wheel_thickness}"/>
+      </geometry>
+      <material name="black"/>
+    </visual>
+    <collision>
+      <origin xyz="0 0 0" rpy="0 0 0"/>
+      <geometry>
+        <cylinder radius="${wheel_radius}" length="${wheel_thickness}"/>
+      </geometry>
+    </collision>
+    <xacro:inertial_cylinder mass="${wheel_mass}" length="${wheel_thickness}" radius="${wheel_radius}">
+      <origin xyz="0 0 0" rpy="0 0 0"/>
+    </xacro:inertial_cylinder>
+  </link>
+  <gazebo reference="back_right_wheel">
+    <material>Gazebo/Black</material>
+  </gazebo>
+  <gazebo>
+    <plugin filename="libgazebo_ros_diff_drive.so" name="differential_drive_controller">
+      <update_rate>100</update_rate>
+      <ros>
+        <namespace>/leader</namespace>
+      </ros>
+      <num_wheel_pairs>2</num_wheel_pairs>
+      <left_joint>front_left_wheel_joint</left_joint>
+      <right_joint>front_right_wheel_joint</right_joint>
+      <left_joint>back_left_wheel_joint</left_joint>
+      <right_joint>back_right_wheel_joint</right_joint>
+      <wheel_separation>0.22</wheel_separation>
+      <wheel_separation>0.22</wheel_separation>
+      <wheel_diameter>0.021</wheel_diameter>
+      <wheel_diameter>0.021</wheel_diameter>
+      <max_wheel_torque>20</max_wheel_torque>
+      <max_wheel_acceleration>1.0</max_wheel_acceleration>
+      <publish_odom>true</publish_odom>
+      <publish_odom_tf>true</publish_odom_tf>
+      <publish_wheel_tf>true</publish_wheel_tf>
+      <use_stamped_vel>false</use_stamped_vel>
+      <odometry_frame>odom</odometry_frame>
+      <robot_base_frame>leader/base_link</robot_base_frame>
+    </plugin>
+  </gazebo>
 </robot>

Commit message: Add C++ follow_target node + update simulation and controllers

File: src/diffbot_sim/urdf/leader.urdf.xacro (robot description, xacro)
@@ -28,7 +28,7 @@
     </inertial>
   </xacro:macro>
-  <xacro:property name="chassis_length" value="0.2"/>
+  <xacro:property name="chassis_length" value="0.25"/>
   <xacro:property name="chassis_width"  value="0.2"/>
-  <xacro:property name="chassis_height" value="0.11"/>
+  <xacro:property name="chassis_height" value="0.14"/>
   <xacro:property name="wheel_radius"    value="0.021"/>
   <xacro:property name="wheel_thickness" value="0.02"/>
@@ -45,6 +45,6 @@
     <color rgba="1 0.3 0.1 1"/>
   </material>
-  <material name="blue">
-    <color rgba="0.2 0.2 1 1"/>
+  <material name="green">
+    <color rgba="0 1 0 1"/>
   </material>
   <material name="black">
@@ -58,5 +58,5 @@
     <parent link="base_link"/>
     <child link="base_footprint"/>
-    <origin xyz="0 0 -0.097" rpy="0 0 0"/>
+    <origin xyz="0 0 -0.121" rpy="0 0 0"/>
   </joint>
   <link name="base_footprint"/>
@@ -68,29 +68,23 @@
   <link name="chassis">
     <visual>
-      <origin xyz="0.07 0 -0.01" rpy="0 0 0"/>
-      <geometry>
-        <box size="0.06 0.2 0.09"/>
-      </geometry>
-      <material name="blue"/>
-    </visual>
-    <visual>
-      <origin xyz="-0.03 0 0" rpy="0 0 0"/>
-      <geometry>
-        <box size="0.14 0.2 0.11"/>
-      </geometry>
-      <material name="blue"/>
-    </visual>
-    <collision>
       <origin xyz="0 0 0" rpy="0 0 0"/>
       <geometry>
         <box size="${chassis_length} ${chassis_width} ${chassis_height}"/>
       </geometry>
-    </collision>
-    <xacro:inertial_box mass="1.0" x="${chassis_length}" y="${chassis_width}" z="${chassis_height}">
-      <origin xyz="0 0 0" rpy="0 0 0"/>
+      <material name="green"/>
+    </visual>
+    <collision>
+      <origin xyz="0 0 0"/>
+      <geometry>
+        <box size="${chassis_length} ${chassis_width} ${chassis_height}"/>
+      </geometry>
+    </collision>
+    <xacro:inertial_box mass="1.0"
+      x="${chassis_length}" y="${chassis_width}" z="${chassis_height}">
+      <origin xyz="0 0 0"/>
     </xacro:inertial_box>
   </link>
   <gazebo reference="chassis">
-    <material>Gazebo/Blue</material>
+    <material>Gazebo/Green</material>
   </gazebo>
   <joint name="front_left_wheel_joint" type="continuous">
